Commit message: new g7_openarm_model

File: models/g7_openarm/origin/g7_openarm.urdf (robot description, URDF)
Before this commit: robot g7_openarm, 31 links, 30 joints
Links:
- link AMR_FLW_link: geometry collision cylinder length=0.075 radius=0.052; visual mesh filename=../meshes/AMR_FLW_link.stl
- link AMR_FL_link: geometry visual mesh filename=../meshes/AMR_FL_link.stl
- link AMR_FRW_link: geometry collision cylinder length=0.075 radius=0.052; visual mesh filename=../meshes/AMR_FRW_link.stl
- link AMR_FR_link: geometry visual mesh filename=../meshes/AMR_FR_link.stl
- link AMR_RLW_link: geometry collision cylinder length=0.075 radius=0.052; visual mesh filename=../meshes/AMR_RLW_link.stl
- link AMR_RL_link: geometry visual mesh filename=../meshes/AMR_RL_link.stl
- link AMR_RRW_link: geometry collision cylinder length=0.075 radius=0.052; visual mesh filename=../meshes/AMR_RRW_link.stl
- link AMR_RR_link: geometry visual mesh filename=../meshes/AMR_RR_link.stl
- link AMR_base_link: geometry collision mesh filename=../meshes/AMR_base_link_collision.stl; visual mesh filename=../meshes/AMR_base_link.stl
- link L_link1: geometry collision mesh filename=../meshes/shoulder_L_link_collision.stl; visual mesh filename=../meshes/L_link1.stl
- link L_link2: geometry visual mesh filename=../meshes/L_link2.stl
- link L_link3: geometry collision mesh filename=../meshes/upper_arm_L_link_collision.stl; visual mesh filename=../meshes/L_link3.stl
- link L_link4: geometry collision mesh filename=../meshes/lower_arm_L_link_collision.stl; visual mesh filename=../meshes/L_link4.stl
- link L_link5: geometry collision mesh filename=../meshes/wrist1_L_link_collision.stl; visual mesh filename=../meshes/L_link5.stl
- link L_link6: geometry collision mesh filename=../meshes/L_link6_collision.stl; visual mesh filename=../meshes/L_link6.stl
- link L_link7: geometry collision mesh filename=../meshes/L_link7_collision.stl; visual mesh filename=../meshes/L_link7.stl
- link L_link8_L: geometry collision mesh filename=../meshes/L_link8_L_collision.stl; visual mesh filename=../meshes/L_link8_L.stl
- link L_link8_R: geometry collision mesh filename=../meshes/L_link8_R_collision.stl; visual mesh filename=../meshes/L_link8_R.stl
- link R_link1: geometry collision mesh filename=../meshes/shoulder_R_link_collision.stl; visual mesh filename=../meshes/R_link1.stl
- link R_link2: geometry visual mesh filename=../meshes/R_link2.stl
- link R_link3: geometry collision mesh filename=../meshes/upper_arm_L_link_collision.stl; visual mesh filename=../meshes/R_link3.stl
- link R_link4: geometry collision mesh filename=../meshes/lower_arm_L_link_collision.stl; visual mesh filename=../meshes/R_link4.stl
- link R_link5: geometry collision mesh filename=../meshes/wrist1_L_link_collision.stl; visual mesh filename=../meshes/R_link5.stl
- link R_link6: geometry collision mesh filename=../meshes/L_link6_collision.stl; visual mesh filename=../meshes/R_link6.stl
- link R_link7: geometry collision mesh filename=../meshes/R_link7_collision.stl; visual mesh filename=../meshes/R_link7.stl
- link R_link8_L: geometry collision mesh filename=../meshes/R_link8_L_collision.stl; visual mesh filename=../meshes/R_link8_L.stl
- link R_link8_R: geometry collision mesh filename=../meshes/R_link8_R_collision.stl; visual mesh filename=../meshes/R_link8_R.stl
- link chest_link: geometry collision mesh filename=../meshes/chest_link_collision.stl; visual mesh filename=../meshes/chest_link.stl
- link openarm_base_link: geometry collision mesh filename=../meshes/openarm_base_link_collision.stl; visual mesh filename=../meshes/openarm_base_link.stl
Joints:
- joint AMR_FLW_joint: limit lower=-1000000.0 upper=1000000.0 effort=15 velocity=10 -> effort=15 velocity=10; type revolute -> continuous
- joint AMR_FRW_joint: limit lower=-1000000.0 upper=1000000.0 effort=15 velocity=10 -> effort=15 velocity=10; type revolute -> continuous
- joint AMR_RLW_joint: limit lower=-1000000.0 upper=1000000.0 effort=15 velocity=10 -> effort=15 velocity=10; type revolute -> continuous
- joint AMR_RRW_joint: limit lower=-1000000.0 upper=1000000.0 effort=15 velocity=10 -> effort=15 velocity=10; type revolute -> continuous
