Commit message: fix axis direction

File: models/g7_openarm/g7_openarm.urdf (robot description, URDF)
Before this commit: robot g7_openarm, 31 links, 30 joints
Joints:
- joint R_2_joint: axis 1 0 0 -> -1 0 0; limit lower=-3.3161253267948965 upper=0.17453267320510335 effort=40 velocity=16.754666 -> lower=-0.17453267320510335 upper=3.3161253267948965 effort=40 velocity=16.754666

File: models/g7_openarm/origin/g7_openarm.urdf (robot description, URDF)
Before this commit: robot g7_openarm, 31 links, 30 joints
Joints:
- joint R_2_joint: axis 1 0 0 -> -1 0 0; limit lower=-3.3161253267948965 upper=0.17453267320510335 effort=40 velocity=16.754666 -> lower=-0.17453267320510335 upper=3.3161253267948965 effort=40 velocity=16.754666

Commit message: latest model (with HEAD)

File: models/g7_openarm/g7_openarm.urdf (robot description, URDF)
Before this commit: robot g7_openarm, 31 links, 30 joints
Links:
- added link HEAD_base_link, mass 0.0288553383340636; collision mesh filename=meshes/base_link.STL; visual mesh filename=meshes/base_link.STL
- added link HEAD_camera_link
- added link HEAD_camera_optical_frame
- added link HEAD_eye_link, mass 0.10791; collision mesh filename=meshes/eye_Link.STL; visual mesh filename=meshes/eye_Link.STL
- added link HEAD_pitch_link, mass 0.180865339049976; collision mesh filename=meshes/pitch_Link.STL; visual mesh filename=meshes/pitch_Link.STL
- added link HEAD_yaw_link, mass 0.21377; collision mesh filename=meshes/yaw_Link.STL; visual mesh filename=meshes/yaw_Link.STL
Joints:
- added joint HEAD_camera_mount_joint: type fixed, parent HEAD_eye_link, child HEAD_camera_link, origin xyz=0 0 0 rpy=0 0 0
- added joint HEAD_camera_optical_joint: type fixed, parent HEAD_camera_link, child HEAD_camera_optical_frame, origin xyz=0 0 0 rpy=-1.57079632679 0 -1.57079632679
- added joint HEAD_eye_joint: type fixed, parent HEAD_pitch_link, child HEAD_eye_link, origin xyz=0.079703 -0.023818 0.0031558 rpy=0 0 0, axis 0 0 0
- added joint HEAD_mount_joint: type fixed, parent chest_link, child HEAD_base_link, origin xyz=0 0 0.063 rpy=0 0 0
- added joint HEAD_pitch_joint: type revolute, parent HEAD_yaw_link, child HEAD_pitch_link, origin xyz=0 0.02775 0.0385 rpy=0 0 0, axis 0 -1 0, limit lower=-3.1415926535897931 upper=3.1415926535897931 effort=5 velocity=2.0
- added joint HEAD_yaw_joint: type revolute, parent HEAD_base_link, child HEAD_yaw_link, origin xyz=0 0 0.06 rpy=0 0 0, axis 0 0 1, limit lower=-1.5707963267948966 upper=1.5707963267948966 effort=5 velocity=2.0
- joint AMR_FLW_joint: limit lower=-1000000.0 upper=1000000.0 effort=15 velocity=10 -> lower=-1000000 upper=1000000 effort=15 velocity=10
- joint AMR_FRW_joint: limit lower=-1000000.0 upper=1000000.0 effort=15 velocity=10 -> lower=-1000000 upper=1000000 effort=15 velocity=10
- joint AMR_RLW_joint: limit lower=-1000000.0 upper=1000000.0 effort=15 velocity=10 -> lower=-1000000 upper=1000000 effort=15 velocity=10
- joint AMR_RRW_joint: limit lower=-1000000.0 upper=1000000.0 effort=15 velocity=10 -> lower=-1000000 upper=1000000 effort=15 velocity=10

Commit message: add HEAD camera and color links with fixed joints

File: models/g7_openarm/g7_openarm.urdf (robot description, URDF)
Before this commit: robot g7_openarm, 37 links, 36 joints
Links:
- added link HEAD_color_link
- added link HEAD_color_optical_frame
- added link HEAD_infra2_link
- added link HEAD_infra2_optical_frame
Joints:
- added joint HEAD_color_mount_joint: type fixed, parent HEAD_camera_link, child HEAD_color_link, origin xyz=0 -0.015 0 rpy=0 0 0
- added joint HEAD_color_optical_joint: type fixed, parent HEAD_color_link, child HEAD_color_optical_frame, origin xyz=0 0 0 rpy=-1.57079632679 0 -1.57079632679
- added joint HEAD_infra2_mount_joint: type fixed, parent HEAD_camera_link, child HEAD_infra2_link, origin xyz=0 0.05 0 rpy=0 0 0
- added joint HEAD_infra2_optical_joint: type fixed, parent HEAD_infra2_link, child HEAD_infra2_optical_frame, origin xyz=0 0 0 rpy=-1.57079632679 0 -1.57079632679
- joint HEAD_camera_mount_joint: origin xyz=0 0 0 rpy=0 0 0 -> xyz=0.0009 0.0135 0 rpy=0 0 0
